File: pcb/robot.sch (KiCad schematic (older format))
At the start: 16 parts, among them J1 MA, J2 MB, J3 Conn_01x03, J4 Conn_01x03, J5 BATT, J6 BATT, J7 STBY, J8 PWR 5V, J9 PWR 3V3, U1 TB6612FNG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

Commit message: updates
Parts:
- removed C1, C2: CP, Capacitors_THT:CP_Radial_D5.0mm_P2.00mm, symbol CP
- removed C3: C_Small, Capacitors_THT:C_Disc_D3.8mm_W2.6mm_P2.50mm, symbol C_Small
- removed J3, J4: Conn_01x03, Pin_Headers:Pin_Header_Straight_1x03_Pitch2.54mm, symbol Conn_01x03
- removed J5, J6: BATT, Pin_Headers:Pin_Header_Straight_1x02_Pitch2.54mm, symbol Conn_01x02
- removed J7: STBY, Pin_Headers:Pin_Header_Straight_1x02_Pitch2.54mm, symbol Conn_01x02
- removed J8: PWR 5V, Pin_Headers:Pin_Header_Straight_1x02_Pitch2.54mm, symbol Conn_01x02
- removed J9: PWR 3V3, Pin_Headers:Pin_Header_Straight_1x02_Pitch2.54mm, symbol Conn_01x02
- added C1, C2: 0.1uF, Capacitors_THT:C_Disc_D3.8mm_W2.6mm_P2.50mm, symbol C_Small
- added C3: 10uF, Capacitors_THT:CP_Radial_D5.0mm_P2.00mm, symbol CP
- added C6: 33uF, Capacitors_THT:CP_Radial_D5.0mm_P2.00mm, symbol CP
- added D1: PWR, LEDs:LED_D3.0mm, symbol LED
- added D2: STBY, LEDs:LED_D3.0mm, symbol LED
- added J11: MB CTRL, Pin_Headers:Pin_Header_Straight_1x02_Pitch2.54mm, symbol Conn_01x02
- added J12: MA CTRL, Pin_Headers:Pin_Header_Straight_1x02_Pitch2.54mm, symbol Conn_01x02
- added J3: Power Connector, Pin_Headers:Pin_Header_Straight_2x05_Pitch2.54mm, symbol Conn_02x05_Counter_Clockwise
- added J4: BATT, Pin_Headers:Pin_Header_Straight_1x02_Pitch2.54mm, symbol Conn_01x02
- added J7: STBY, Pin_Headers:Pin_Header_Straight_1x03_Pitch2.54mm, symbol Conn_01x03
- added J8: PWR, Pin_Headers:Pin_Header_Straight_1x03_Pitch2.54mm, symbol Conn_01x03
- added Q1, Q2: PN2222A, TO_SOT_Packages_THT:TO-92_Inline_Narrow_Oval, symbol PN2222A
- added R1, R2: 330, Resistors_THT:R_Axial_DIN0204_L3.6mm_D1.6mm_P5.08mm_Horizontal, symbol R_Small
- added R3, R4, R5, R6: 10k, Resistors_THT:R_Axial_DIN0204_L3.6mm_D1.6mm_P5.08mm_Horizontal, symbol R_Small
- C4: value C_Small -> 0.1uF
- J1: value MA -> MA PWR
- J2: value MB -> MB PWR
Connections:
- net labels added: A1, A2, APWM, B1, B2, BPWM, VCC
- wire segments 71 -> 112
- no-connect marks 0 -> 1
Other:
- note added: "Dual Motor Driver\nContinous: 1.2A\nPeak: 3A"
- note added: "Motor Power 5V"
- note added: "Power Switch"
- note added: "add:\npwr led\nsecond to-220?\ndoes to-92 provide 750mA or 500 mA?\ntransistor not on MD to simplify interface"
- moved on the sheet: C4, J1, J2, U1, U2, U3
