File: pcb-v2/robot.kicad_pcb (KiCad board)
At the start: 2 copper layers, 34.9 x 69.2 mm, 30 parts, among them J1 M1 PWR, J11 MB CTRL, J12 MA CTRL, J2 M2 PWR, J3 Power Connector, J4 BATT, J7 STBY, J8 PWR, Q1 PN2222A, Q2 PN2222A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

Commit message: up
Parts:
- removed D2: STBY, LEDs:LED_D3.0mm
- removed J8: PWR, Pin_Headers:Pin_Header_Straight_1x03_Pitch2.54mm
- removed R2: 330, Resistors_THT:R_Axial_DIN0204_L3.6mm_D1.6mm_P5.08mm_Horizontal
- removed U1: TB6612FNG, kevin:Adafruit_Motor_Driver_TB6612
- added J5: TB6612_Motor_Driver, bob:Pololu_TB6612, F.Cu at (106.0, 57.8)
- added J6: STBY, Pin_Headers:Pin_Header_Straight_1x02_Pitch2.54mm, F.Cu at (99.7, 79.4)
- J7: value STBY -> PWR; footprint Pin_Headers:Pin_Header_Straight_1x03_Pitch2.54mm -> Pin_Headers:Pin_Header_Straight_1x02_Pitch2.54mm
- moved J7 38.9 mm to (108.6, 54.6), turned to 90 degrees
- moved R1 30.8 mm to (98.4, 48.3), turned to 90 degrees
- moved J2 29.9 mm to (128.3, 63.5), turned to 0 degrees
- moved J4 25.0 mm to (120.0, 54.6), turned to 270 degrees
- moved Q1 21.9 mm to (102.9, 49.5), turned to 0 degrees
- moved C2 19.8 mm to (106.0, 32.4)
- moved R6 18.5 mm to (116.2, 63.5)
- moved R5 17.7 mm to (111.8, 63.5)
- moved R3 11.7 mm to (111.8, 73.0), turned to 90 degrees
- moved J11 7.75 mm to (99.1, 87.0), turned to 90 degrees
- moved J1 6.98 mm to (128.3, 57.8)
- moved J12 6.84 mm to (125.1, 87.0), turned to 90 degrees
- moved R4 5.85 mm to (116.2, 67.9), turned to 270 degrees
- moved J3 3.81 mm to (118.1, 89.5)
- moved D1 3.18 mm to (99.1, 69.8), turned to 0 degrees
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Connections:
- J7 pad 1: STBY -> VCC
- J7 pad 2: +3V3 -> +BATT
Other:
- board text added: "aaa bbb bbb bbb bbb"
