File: pcb-v2/robot.sch (KiCad schematic (older format))
At the start: 26 parts, among them J1 M1 PWR, J11 MB CTRL, J12 MA CTRL, J2 M2 PWR, J3 Power Connector, J4 BATT, J5 TB6612_Motor_Driver, J7 STBY, J8 PWR, Q1 PN2222A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

Commit message: up
Parts:
- removed D2: STBY, LEDs:LED_D3.0mm, symbol LED
- removed J7: STBY, Pin_Headers:Pin_Header_Straight_1x03_Pitch2.54mm, symbol Conn_01x03
- removed J8: PWR, Pin_Headers:Pin_Header_Straight_1x03_Pitch2.54mm, symbol Conn_01x03
- removed R2: 330, Resistors_THT:R_Axial_DIN0204_L3.6mm_D1.6mm_P5.08mm_Horizontal, symbol R_Small
- added J6: STBY, Pin_Headers:Pin_Header_Straight_1x02_Pitch2.54mm, symbol Conn_01x02
- added J7: PWR, Pin_Headers:Pin_Header_Straight_1x02_Pitch2.54mm, symbol Conn_01x02
- J5: footprint (none) -> bob:Pololu_TB6612
Connections:
- net +3V3: now also J6.1 (Pin_1)
- net +BATT: now also J7.2 (Pin_2)
- net STBY: now also J6.2 (Pin_2)
- net VCC: now also J7.1 (Pin_1)
- no-connect marks 1 -> 0
