File: pcb-v3/robot.sch (KiCad schematic (older format))
At the start: 23 parts, among them J1 M1 PWR, J11 MB CTRL, J12 MA CTRL, J2 M2 PWR, J3 Power Connector, J4 BATT, J5 TB6612_Motor_Driver, J7 PWR, Q1 PN2222A, Q2 PN2222A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

Commit message: fixed md footprint and 1/4 w resistors
Parts:
- removed Q1, Q2: PN2222A, TO_SOT_Packages_THT:TO-92_Inline_Narrow_Oval, symbol PN2222A
- added Q1, Q2: 2N3904, TO_SOT_Packages_THT:TO-92_Inline_Narrow_Oval, symbol 2N3904
- R1, R3, R4, R5, R6: footprint Resistors_THT:R_Axial_DIN0204_L3.6mm_D1.6mm_P5.08mm_Horizontal -> Resistors_THT:R_Axial_DIN0207_L6.3mm_D2.5mm_P10.16mm_Horizontal
Connections:
- net A1: now also Q2.3 (C)
- net B1: now also Q1.3 (C)
- net GND: now also Q1.1 (E), Q2.1 (E)
- net at R5.2: now also Q1.2 (B)
- net at R6.2: now also Q2.2 (B)
Changed lines of the file:
@@
 F 0 "R1" H 7430 4470 50  0000 L CNN
 F 1 "330" H 7430 4410 50  0000 L CNN
-F 2 "Resistors_THT:R_Axial_DIN0204_L3.6mm_D1.6mm_P5.08mm_Horizontal" H 7400 4450 50  0001 C CNN
+F 2 "Resistors_THT:R_Axial_DIN0207_L6.3mm_D2.5mm_P10.16mm_Horizontal" H 7400 4450 50  0001 C CNN
 F 3 "" H 7400 4450 50  0001 C CNN
 	1    7400 4450
@@
 	6400 3800 6650 3800
 $Comp
-L PN2222A Q1
-U 1 1 5AC80E58
-P 3650 5950
-F 0 "Q1" H 3850 6025 50  0000 L CNN
-F 1 "PN2222A" H 3850 5950 50  0000 L CNN
-F 2 "TO_SOT_Packages_THT:TO-92_Inline_Narrow_Oval" H 3850 5875 50  0001 L CIN
-F 3 "" H 3650 5950 50  0001 L CNN
-	1    3650 5950
-	1    0    0    -1
-$EndComp
-$Comp
-L +5V #PWR015
+L +5V #PWR012
 U 1 1 5AC814AB
 P 3750 5400
-F 0 "#PWR015" H 3750 5250 50  0001 C CNN
+F 0 "#PWR012" H 3750 5250 50  0001 C CNN
 F 1 "+5V" H 3750 5540 50  0000 C CNN
 F 2 "" H 3750 5400 50  0001 C CNN
@@
 F 0 "R3" H 3780 5620 50  0000 L CNN
 F 1 "10k" H 3780 5560 50  0000 L CNN
-F 2 "Resistors_THT:R_Axial_DIN0204_L3.6mm_D1.6mm_P5.08mm_Horizontal" H 3750 5600 50  0001 C CNN
+F 2 "Resistors_THT:R_Axial_DIN0207_L6.3mm_D2.5mm_P10.16mm_Horizontal" H 3750 5600 50  0001 C CNN
 F 3 "" H 3750 5600 50  0001 C CNN
 	1    3750 5600
@@
 B2
 $Comp
-L GND #PWR016
+L GND #PWR013
 U 1 1 5AC81A5E
 P 3750 6250
-F 0 "#PWR016" H 3750 6000 50  0001 C CNN
+F 0 "#PWR013" H 3750 6000 50  0001 C CNN
 F 1 "GND" H 3750 6100 50  0000 C CNN
 F 2 "" H 3750 6250 50  0001 C CNN
@@
 	3250 6050 3000 6050
 $Comp
-L PN2222A Q2
-U 1 1 5AC827C8
-P 4950 7150
-F 0 "Q2" H 5150 7225 50  0000 L CNN
-F 1 "PN2222A" H 5150 7150 50  0000 L CNN
-F 2 "TO_SOT_Packages_THT:TO-92_Inline_Narrow_Oval" H 5150 7075 50  0001 L CIN
-F 3 "" H 4950 7150 50  0001 L CNN
-	1    4950 7150
-	1    0    0    -1
-$EndComp
-$Comp
-L +5V #PWR017
+L +5V #PWR014
 U 1 1 5AC827CE
 P 5050 6600
-F 0 "#PWR017" H 5050 6450 50  0001 C CNN
+F 0 "#PWR014" H 5050 6450 50  0001 C CNN
 F 1 "+5V" H 5050 6740 50  0000 C CNN
 F 2 "" H 5050 6600 50  0001 C CNN
@@
 F 0 "R4" H 5080 6820 50  0000 L CNN
 F 1 "10k" H 5080 6760 50  0000 L CNN
-F 2 "Resistors_THT:R_Axial_DIN0204_L3.6mm_D1.6mm_P5.08mm_Horizontal" H 5050 6800 50  0001 C CNN
+F 2 "Resistors_THT:R_Axial_DIN0207_L6.3mm_D2.5mm_P10.16mm_Horizontal" H 5050 6800 50  0001 C CNN
 F 3 "" H 5050 6800 50  0001 C CNN
 	1    5050 6800
@@
 A2
 $Comp
-L GND #PWR018
+L GND #PWR015
 U 1 1 5AC827E2
 P 5050 7450
-F 0 "#PWR018" H 5050 7200 50  0001 C CNN
+F 0 "#PWR015" H 5050 7200 50  0001 C CNN
 F 1 "GND" H 5050 7300 50  0000 C CNN
 F 2 "" H 5050 7450 50  0001 C CNN
@@
 F 0 "R6" H 4580 7170 50  0000 L CNN
 F 1 "10k" H 4580 7110 50  0000 L CNN
-F 2 "Resistors_THT:R_Axial_DIN0204_L3.6mm_D1.6mm_P5.08mm_Horizontal" H 4550 7150 50  0001 C CNN
+F 2 "Resistors_THT:R_Axial_DIN0207_L6.3mm_D2.5mm_P10.16mm_Horizontal" H 4550 7150 50  0001 C CNN
 F 3 "" H 4550 7150 50  0001 C CNN
 	1    4550 7150
@@
 F 0 "R5" H 3280 5970 50  0000 L CNN
 F 1 "10k" H 3280 5910 50  0000 L CNN
-F 2 "Resistors_THT:R_Axial_DIN0204_L3.6mm_D1.6mm_P5.08mm_Horizontal" H 3250 5950 50  0001 C CNN
+F 2 "Resistors_THT:R_Axial_DIN0207_L6.3mm_D2.5mm_P10.16mm_Horizontal" H 3250 5950 50  0001 C CNN
 F 3 "" H 3250 5950 50  0001 C CNN
 	1    3250 5950
@@
 $EndComp
 $Comp
-L +5V #PWR019
+L +5V #PWR016
 U 1 1 5ACA8D25
 P 2700 1600
-F 0 "#PWR019" H 2700 1450 50  0001 C CNN
+F 0 "#PWR016" H 2700 1450 50  0001 C CNN
 F 1 "+5V" H 2700 1740 50  0000 C CNN
 F 2 "" H 2700 1600 50  0001 C CNN
@@
 $EndComp
 $Comp
-L +3V3 #PWR020
+L +3V3 #PWR017
 U 1 1 5ACA94EC
 P 2850 1500
-F 0 "#PWR020" H 2850 1350 50  0001 C CNN
+F 0 "#PWR017" H 2850 1350 50  0001 C CNN
 F 1 "+3V3" H 2850 1640 50  0000 C CNN
 F 2 "" H 2850 1500 50  0001 C CNN
@@
 $EndComp
 $Comp
-L GND #PWR021
+L GND #PWR018
 U 1 1 5ACA9BA5
 P 3800 1850
-F 0 "#PWR021" H 3800 1600 50  0001 C CNN
+F 0 "#PWR018" H 3800 1600 50  0001 C CNN
 F 1 "GND" H 3800 1700 50  0000 C CNN
 F 2 "" H 3800 1850 50  0001 C CNN
@@
 Connection ~ 3000 1300
 $Comp
-L +3V3 #PWR022
+L +3V3 #PWR019
 U 1 1 5ACAB044
 P 7400 3750
-F 0 "#PWR022" H 7400 3600 50  0001 C CNN
+F 0 "#PWR019" H 7400 3600 50  0001 C CNN
 F 1 "+3V3" H 7400 3890 50  0000 C CNN
 F 2 "" H 7400 3750 50  0001 C CNN
@@
 $EndComp
 $Comp
-L +5V #PWR023
+L +5V #PWR020
 U 1 1 5ACB0D91
 P 6650 3700
-F 0 "#PWR023" H 6650 3550 50  0001 C CNN
+F 0 "#PWR020" H 6650 3550 50  0001 C CNN
 F 1 "+5V" H 6650 3840 50  0000 C CNN
 F 2 "" H 6650 3700 50  0001 C CNN
@@
 $EndComp
 $Comp
-L +5V #PWR024
+L +5V #PWR021
 U 1 1 5ACB1407
 P 5850 2000
-F 0 "#PWR024" H 5850 1850 50  0001 C CNN
+F 0 "#PWR021" H 5850 1850 50  0001 C CNN
 F 1 "+5V" H 5850 2140 50  0000 C CNN
 F 2 "" H 5850 2000 50  0001 C CNN
@@
 $EndComp
 $Comp
-L +5V #PWR025
+L +5V #PWR022
 U 1 1 5ACB2641
 P 5450 5250
-F 0 "#PWR025" H 5450 5100 50  0001 C CNN
+F 0 "#PWR022" H 5450 5100 50  0001 C CNN
 F 1 "+5V" H 5450 5390 50  0000 C CNN
 F 2 "" H 5450 5250 50  0001 C CNN
@@
 $EndComp
 $Comp
-L GND #PWR026
+L GND #PWR023
 U 1 1 5ACB9CCB
 P 4850 1350
-F 0 "#PWR026" H 4850 1100 50  0001 C CNN
+F 0 "#PWR023" H 4850 1100 50  0001 C CNN
 F 1 "GND" H 4850 1200 50  0000 C CNN
 F 2 "" H 4850 1350 50  0001 C CNN
@@
 	5700 2550 5650 2550
 $Comp
-L +BATT #PWR028
+L +BATT #PWR024
 U 1 1 5AD3E29C
 P 5500 3700
-F 0 "#PWR028" H 5500 3550 50  0001 C CNN
+F 0 "#PWR024" H 5500 3550 50  0001 C CNN
 F 1 "+BATT" H 5500 3840 50  0000 C CNN
 F 2 "" H 5500 3700 50  0001 C CNN
@@
 $EndComp
 $Comp
-L +BATT #PWR029
+L +BATT #PWR025
 U 1 1 5AD3F3B7
 P 3000 1300
-F 0 "#PWR029" H 3000 1150 50  0001 C CNN
+F 0 "#PWR025" H 3000 1150 50  0001 C CNN
 F 1 "+BATT" H 3000 1440 50  0000 C CNN
 F 2 "" H 3000 1300 50  0001 C CNN
@@
 	3150 1500 2850 1500
 $Comp
-L +5V #PWR?
+L +5V #PWR026
 U 1 1 5AD44078
 P 7650 2300
-F 0 "#PWR?" H 7650 2150 50  0001 C CNN
+F 0 "#PWR026" H 7650 2150 50  0001 C CNN
 F 1 "+5V" H 7650 2440 50  0000 C CNN
 F 2 "" H 7650 2300 50  0001 C CNN
@@
 Wire Wire Line
 	7650 2350 7650 2300
+$Comp
+L 2N3904 Q1
+U 1 1 5AD4E8D0
+P 3650 5950
+F 0 "Q1" H 3850 6025 50  0000 L CNN
+F 1 "2N3904" H 3850 5950 50  0000 L CNN
+F 2 "TO_SOT_Packages_THT:TO-92_Inline_Narrow_Oval" H 3850 5875 50  0001 L CIN
+F 3 "" H 3650 5950 50  0001 L CNN
+	1    3650 5950
+	1    0    0    -1
+$EndComp
+$Comp
+L 2N3904 Q2
+U 1 1 5AD4EECC
+P 4950 7150
+F 0 "Q2" H 5150 7225 50  0000 L CNN
+F 1 "2N3904" H 5150 7150 50  0000 L CNN
+F 2 "TO_SOT_Packages_THT:TO-92_Inline_Narrow_Oval" H 5150 7075 50  0001 L CIN
+F 3 "" H 4950 7150 50  0001 L CNN
+	1    4950 7150
+	1    0    0    -1
+$EndComp
 $EndSCHEMATC
