File: pcb-v3/robot.kicad_pcb (KiCad board)
At the start: 2 copper layers, 34.9 x 69.2 mm, 27 parts, among them J1 M1 PWR, J11 MB CTRL, J12 MA CTRL, J2 M2 PWR, J3 Power Connector, J4 BATT, J5 TB6612_Motor_Driver, J7 PWR, Q1 PN2222A, Q2 PN2222A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

Commit message: fixed md footprint and 1/4 w resistors
Parts:
- Q1, Q2: value PN2222A -> 2N3904
- R1, R3, R4, R5, R6: footprint Resistors_THT:R_Axial_DIN0204_L3.6mm_D1.6mm_P5.08mm_Horizontal -> Resistors_THT:R_Axial_DIN0207_L6.3mm_D2.5mm_P10.16mm_Horizontal
- moved R5 4.84 mm to (127.0, 68.6)
- moved R1 3.24 mm to (99.7, 87.0)
- moved R4 2.69 mm to (127.6, 53.3)
- moved R6 2.29 mm to (127.0, 66.0)
- moved R3 2.01 mm to (114.3, 70.5)
- moved J5 1.42 mm to (106.7, 60.3)
- moved Q1 0.90 mm to (122.6, 83.2)
- moved U3 0.64 mm to (112.4, 83.2)
Routing:
- net B2: track 23.6 -> 29.6 mm
- net +5V: track 103.0 -> 97.2 mm
- net A2: track 38.5 -> 43.7 mm, vias 1 -> 2
- net Net-(Q1-Pad2): track 6.13 -> 8.30 mm
- net Net-(D1-Pad1): track 4.71 -> 6.66 mm
- net A1: track 17.7 -> 19.4 mm
- net Net-(J2-Pad2): track 5.08 -> 6.61 mm
- net Net-(J2-Pad1): track 5.08 -> 6.61 mm
- net Net-(J1-Pad1): track 6.66 -> 8.19 mm
- net Net-(J1-Pad2): track 6.66 -> 8.19 mm
- net +BATT: track 75.8 -> 74.8 mm
- net GND: track 132.3 -> 133.2 mm, vias 0 -> 1
- net B1: track 19.2 -> 18.6 mm
- net BPWM: track 20.1 -> 20.7 mm, vias 0 -> 1
- net APWM: track 39.6 -> 39.9 mm, vias 1 -> 2

Commit message: small fixes
Parts:
- added ?: , Symbols:OSHW-Logo_5.7x6mm_SilkScreen, F.Cu at (123.2, 35.6)
- U3: value L78L33_TO92 -> L78L33
Other:
- board text added: "1"
- board text added: "GND"
- board text added: "Walchko (c) 2018"
